File: smart-pedal/smart-pedal/smart-pedal.sch (EAGLE design)
At the start: 18 parts, among them Q1 MMBT5088

Commit message: cleanup
Changed lines of the file:
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@@
 <pinref part="U$2" gate="G$1" pin="VIN"/>
 <wire x1="38.1" y1="-55.88" x2="48.26" y2="-55.88" width="0.1524" layer="91"/>
+<label x="48.26" y="-58.42" size="1.778" layer="95"/>
 </segment>
 </net>
